File: pcb/SD_GPS_sub-board.sch (KiCad schematic (older format))
At the start: 7 parts, among them J5 Conn_02x05_Odd_Even, J6 Micro_SD_Card, J7 U.FL-R-SMT-101, U9 MAX-M8W

Commit message: Board: use different USB-C Receptable
Parts:
- R18: footprint Resistor_SMD:R_0201_0603Metric -> Resistor_SMD:R_0402_1005Metric
Changed lines of the file:
@@
 F 0 "R18" V 1743 3300 50  0000 C CNN
 F 1 "10R" V 1834 3300 50  0000 C CNN
-F 2 "Resistor_SMD:R_0201_0603Metric" V 1880 3300 50  0001 C CNN
+F 2 "Resistor_SMD:R_0402_1005Metric" V 1880 3300 50  0001 C CNN
 F 3 "~" H 1950 3300 50  0001 C CNN
 	1    1950 3300
