File: pcb/obd32.sch (KiCad schematic (older format))
At the start: 61 parts, among them J1 USB_C_Receptacle_USB2.0, J2 Micro_SD_Card, J3 OBD2, J4 67329-8040, J5 Conn_01x04_Female, SW1 SW_Push, SW2 SW_Push, SW3 SW_Push, U1 LMR33630BDDA, U2 ICM-20689, U3 AZ1117C-3.3, U4 ESP32-WROOM-32, U5 SiP32431DR3, U6 MCP2562-E-MF, U7 BMP280, U8 CP2102N-A01-GQFN24

Commit message: PCB: Move components from bottom to top side of board. Move SD-card slot to sub board. Add SAM-M8N GPS-receiver
Parts:
- removed J2: Micro_SD_Card, Connector_Card:microSD_HC_Hirose_DM3AT-SF-PEJM5, symbol Connector:Micro_SD_Card
- removed J5: Conn_01x04_Female, Connector_PinSocket_2.54mm:PinSocket_1x04_P2.54mm_Vertical_SMD_Pin1Left, symbol Connector:Conn_01x04_Female
- removed U7: BMP280, Package_LGA:Bosch_LGA-8_2x2.5mm_P0.65mm_ClockwisePinNumbering, symbol Sensor_Pressure:BMP280
- added C22: 100nF, Capacitor_SMD:C_0201_0603Metric, symbol Device:C
- added J4: Conn_02x05_Odd_Even, Connector_PinSocket_2.54mm:PinSocket_2x05_P2.54mm_Vertical, symbol Connector_Generic:Conn_02x05_Odd_Even
- added JP2: SolderJumper_2_Open, Jumper:SolderJumper-2_P1.3mm_Open_RoundedPad1.0x1.5mm, symbol Jumper:SolderJumper_2_Open
- added JP4: Jumper_NO_Small, Connector_PinHeader_2.54mm:PinHeader_1x02_P2.54mm_Vertical, symbol Device:Jumper_NO_Small
- added R7: 10K, Resistor_SMD:R_0201_0603Metric, symbol Device:R
- added U6: BMP388, BMP388:BMP388, symbol obd32-rescue:BMP388-BMP388
- C17: renamed from C18; value 0.1µF -> 100nF
- J2: renamed from J1; footprint Connector_USB:USB_C_Receptacle_HRO_TYPE-C-31-M-12 -> Connector_USB:USB_C_Receptacle_GCT_USB4085
- R8: renamed from R1; value 876K -> 866K
- U2: renamed from U4; footprint RF_Module:ESP32-WROOM-32 -> RF_Module:ESP32-WROOM-32U
- renumbered C8 to C10, C6 to C11, C9 to C12, C10 to C13, C15 to C14, C16 to C15, C17 to C16, C13 to C18, C11 to C19, C19 to C2, C14 to C20, C12 to C21, C2 to C3, C3 to C4, C4 to C5, C20 to C6, C5 to C8, C21 to C9, D3 to D1, D4 to D2, D5 to D3, D1 to D4, D2 to D5, J4 to J1, R10 to R1, R7 to R10, R8 to R11, R3 to R12, R4 to R13, R15 to R14, R16 to R15, R17 to R16, R9 to R17, R11 to R2, R5 to R3, R12 to R4, R13 to R5, R14 to R6, R2 to R9, SW2 to SW1, SW1 to SW2, U8 to U4, U2 to U5, U6 to U7, U5 to U8
Connections:
- wire segments 107 -> 105
- no-connect marks 2 -> 19
Other:
- moved on the sheet: C17, C18, C20, R17, R8, R9, U7

Commit message: Board: use different USB-C Receptable
Parts:
- C10, C14, C15, C16, C17, C18, C19, C2, C20, C21, C22, C7, C9: footprint Capacitor_SMD:C_0201_0603Metric -> Capacitor_SMD:C_0402_1005Metric
- J2: footprint Connector_USB:USB_C_Receptacle_GCT_USB4085 -> USB_C_Receptacle_JAE_DX07S016JA1:USB_C_Receptacle_JAE_DX07S016JA1
- R1, R10, R11, R12, R13, R14, R15, R16, R17, R2, R3, R4, R5, R6, R7, R8, R9: footprint Resistor_SMD:R_0201_0603Metric -> Resistor_SMD:R_0402_1005Metric
Changed lines of the file:
@@
 F 0 "R12" H 3030 6604 50  0000 R CNN
 F 1 "100K" H 3030 6695 50  0000 R CNN
-F 2 "Resistor_SMD:R_0201_0603Metric" V 3030 6650 50  0001 C CNN
+F 2 "Resistor_SMD:R_0402_1005Metric" V 3030 6650 50  0001 C CNN
 F 3 "~" H 3100 6650 50  0001 C CNN
 	1    3100 6650
@@
 F 0 "C20" V 10052 2250 50  0000 C CNN
 F 1 "0.1µF" V 9950 2200 50  0000 C CNN
-F 2 "Capacitor_SMD:C_0201_0603Metric" H 9838 2100 50  0001 C CNN
+F 2 "Capacitor_SMD:C_0402_1005Metric" H 9838 2100 50  0001 C CNN
 F 3 "~" H 9800 2250 50  0001 C CNN
 	1    9800 2250
@@
 F 0 "C18" H 8850 3000 50  0000 R CNN
 F 1 "0.1µF" H 8850 3100 50  0000 R CNN
-F 2 "Capacitor_SMD:C_0201_0603Metric" H 8538 2850 50  0001 C CNN
+F 2 "Capacitor_SMD:C_0402_1005Metric" H 8538 2850 50  0001 C CNN
 F 3 "~" H 8500 3000 50  0001 C CNN
 	1    8500 3000
@@
 F 0 "C21" H 10865 5946 50  0000 L CNN
 F 1 "0.1µF" H 10865 5855 50  0000 L CNN
-F 2 "Capacitor_SMD:C_0201_0603Metric" H 10788 5750 50  0001 C CNN
+F 2 "Capacitor_SMD:C_0402_1005Metric" H 10788 5750 50  0001 C CNN
 F 3 "~" H 10750 5900 50  0001 C CNN
 	1    10750 5900
@@
 F 0 "C19" H 9300 5900 50  0000 L CNN
 F 1 "0.1µF" H 9300 5800 50  0000 L CNN
-F 2 "Capacitor_SMD:C_0201_0603Metric" H 9688 5750 50  0001 C CNN
+F 2 "Capacitor_SMD:C_0402_1005Metric" H 9688 5750 50  0001 C CNN
 F 3 "~" H 9650 5900 50  0001 C CNN
 	1    9650 5900
@@
 F 0 "R13" H 3030 6904 50  0000 R CNN
 F 1 "24.9K" H 3030 6995 50  0000 R CNN
-F 2 "Resistor_SMD:R_0201_0603Metric" V 3030 6950 50  0001 C CNN
+F 2 "Resistor_SMD:R_0402_1005Metric" V 3030 6950 50  0001 C CNN
 F 3 "~" H 3100 6950 50  0001 C CNN
 	1    3100 6950
@@
 F 0 "R9" H 1180 7104 50  0000 R CNN
 F 1 "100K" H 1180 7195 50  0000 R CNN
-F 2 "Resistor_SMD:R_0201_0603Metric" V 1180 7150 50  0001 C CNN
+F 2 "Resistor_SMD:R_0402_1005Metric" V 1180 7150 50  0001 C CNN
 F 3 "~" H 1250 7150 50  0001 C CNN
 	1    1250 7150
@@
 F 0 "R8" H 1180 6804 50  0000 R CNN
 F 1 "866K" H 1180 6895 50  0000 R CNN
-F 2 "Resistor_SMD:R_0201_0603Metric" V 1180 6850 50  0001 C CNN
+F 2 "Resistor_SMD:R_0402_1005Metric" V 1180 6850 50  0001 C CNN
 F 3 "~" H 1250 6850 50  0001 C CNN
 	1    1250 6850
@@
 F 0 "R11" H 1780 1154 50  0000 R CNN
 F 1 "27K" H 1780 1245 50  0000 R CNN
-F 2 "Resistor_SMD:R_0201_0603Metric" V 1780 1200 50  0001 C CNN
+F 2 "Resistor_SMD:R_0402_1005Metric" V 1780 1200 50  0001 C CNN
 F 3 "~" H 1850 1200 50  0001 C CNN
 	1    1850 1200
@@
 F 0 "R10" H 1780 854 50  0000 R CNN
 F 1 "100K" H 1780 945 50  0000 R CNN
-F 2 "Resistor_SMD:R_0201_0603Metric" V 1780 900 50  0001 C CNN
+F 2 "Resistor_SMD:R_0402_1005Metric" V 1780 900 50  0001 C CNN
 F 3 "~" H 1850 900 50  0001 C CNN
 	1    1850 900
@@
 F 0 "R17" H 10530 2704 50  0000 R CNN
 F 1 "120R" H 10530 2795 50  0000 R CNN
-F 2 "Resistor_SMD:R_0201_0603Metric" V 10530 2750 50  0001 C CNN
+F 2 "Resistor_SMD:R_0402_1005Metric" V 10530 2750 50  0001 C CNN
 F 3 "~" H 10600 2750 50  0001 C CNN
 	1    10600 2750
@@
 F 0 "R1" V 1300 1500 50  0000 R CNN
 F 1 "4K7" V 1200 1500 50  0000 R CNN
-F 2 "Resistor_SMD:R_0201_0603Metric" V 1030 1400 50  0001 C CNN
+F 2 "Resistor_SMD:R_0402_1005Metric" V 1030 1400 50  0001 C CNN
 F 3 "~" H 1100 1400 50  0001 C CNN
 	1    1100 1400
@@
 F 0 "R2" V 1200 1500 50  0000 R CNN
 F 1 "4K7" V 1300 1550 50  0000 R CNN
-F 2 "Resistor_SMD:R_0201_0603Metric" V 1030 1500 50  0001 C CNN
+F 2 "Resistor_SMD:R_0402_1005Metric" V 1030 1500 50  0001 C CNN
 F 3 "~" H 1100 1500 50  0001 C CNN
 	1    1100 1500
@@
 F 0 "C16" H 6800 2600 50  0000 L CNN
 F 1 "0.1µF" H 6700 2500 50  0000 L CNN
-F 2 "Capacitor_SMD:C_0201_0603Metric" H 7038 2250 50  0001 C CNN
+F 2 "Capacitor_SMD:C_0402_1005Metric" H 7038 2250 50  0001 C CNN
 F 3 "~" H 7000 2400 50  0001 C CNN
 	1    7000 2400
@@
 F 0 "C14" V 5950 3400 50  0000 L CNN
 F 1 "10nF" V 5850 3300 50  0000 L CNN
-F 2 "Capacitor_SMD:C_0201_0603Metric" H 5788 3100 50  0001 C CNN
+F 2 "Capacitor_SMD:C_0402_1005Metric" H 5788 3100 50  0001 C CNN
 F 3 "~" H 5750 3250 50  0001 C CNN
 	1    5750 3250
@@
 F 0 "C15" H 6500 3450 50  0000 L CNN
 F 1 "0.47µF" H 6400 3350 50  0000 L CNN
-F 2 "Capacitor_SMD:C_0201_0603Metric" H 6438 3300 50  0001 C CNN
+F 2 "Capacitor_SMD:C_0402_1005Metric" H 6438 3300 50  0001 C CNN
 F 3 "~" H 6400 3450 50  0001 C CNN
 	1    6400 3450
@@
 F 0 "R3" H 1080 2054 50  0000 R CNN
 F 1 "10K" H 1080 2145 50  0000 R CNN
-F 2 "Resistor_SMD:R_0201_0603Metric" V 1080 2100 50  0001 C CNN
+F 2 "Resistor_SMD:R_0402_1005Metric" V 1080 2100 50  0001 C CNN
 F 3 "~" H 1150 2100 50  0001 C CNN
 	1    1150 2100
@@
 F 0 "R4" V 943 3650 50  0000 C CNN
 F 1 "65R" V 1034 3650 50  0000 C CNN
-F 2 "Resistor_SMD:R_0201_0603Metric" V 1080 3650 50  0001 C CNN
+F 2 "Resistor_SMD:R_0402_1005Metric" V 1080 3650 50  0001 C CNN
 F 3 "~" H 1150 3650 50  0001 C CNN
 	1    1150 3650
@@
 F 0 "R5" V 943 4000 50  0000 C CNN
 F 1 "65R" V 1034 4000 50  0000 C CNN
-F 2 "Resistor_SMD:R_0201_0603Metric" V 1080 4000 50  0001 C CNN
+F 2 "Resistor_SMD:R_0402_1005Metric" V 1080 4000 50  0001 C CNN
 F 3 "~" H 1150 4000 50  0001 C CNN
 	1    1150 4000
@@
 F 0 "R6" V 943 4350 50  0000 C CNN
 F 1 "5R" V 1034 4350 50  0000 C CNN
-F 2 "Resistor_SMD:R_0201_0603Metric" V 1080 4350 50  0001 C CNN
+F 2 "Resistor_SMD:R_0402_1005Metric" V 1080 4350 50  0001 C CNN
 F 3 "~" H 1150 4350 50  0001 C CNN
 	1    1150 4350
@@
 F 0 "J2" H 7057 6067 50  0000 C CNN
 F 1 "USB_C_Receptacle_USB2.0" H 7057 5976 50  0000 C CNN
-F 2 "Connector_USB:USB_C_Receptacle_GCT_USB4085" H 7100 5200 50  0001 C CNN
+F 2 "USB_C_Receptacle_JAE_DX07S016JA1:USB_C_Receptacle_JAE_DX07S016JA1" H 7100 5200 50  0001 C CNN
 F 3 "https://www.usb.org/sites/default/files/documents/usb_type-c.zip" H 7100 5200 50  0001 C CNN
 	1    6950 5200
@@
 F 0 "R15" V 8050 4700 50  0000 C CNN
 F 1 "5.1K" V 8050 4900 50  0000 C CNN
-F 2 "Resistor_SMD:R_0201_0603Metric" V 8080 4800 50  0001 C CNN
+F 2 "Resistor_SMD:R_0402_1005Metric" V 8080 4800 50  0001 C CNN
 F 3 "~" H 8150 4800 50  0001 C CNN
 	1    8150 4800
@@
 F 0 "R16" V 8050 5000 50  0000 C CNN
 F 1 "5.1K" V 8050 4800 50  0000 C CNN
-F 2 "Resistor_SMD:R_0201_0603Metric" V 8080 4900 50  0001 C CNN
+F 2 "Resistor_SMD:R_0402_1005Metric" V 8080 4900 50  0001 C CNN
 F 3 "~" H 8150 4900 50  0001 C CNN
 	1    8150 4900
@@
 F 0 "R14" H 4130 4354 50  0000 R CNN
 F 1 "1K" H 4130 4445 50  0000 R CNN
-F 2 "Resistor_SMD:R_0201_0603Metric" V 4130 4400 50  0001 C CNN
+F 2 "Resistor_SMD:R_0402_1005Metric" V 4130 4400 50  0001 C CNN
 F 3 "~" H 4200 4400 50  0001 C CNN
 	1    4200 4400
@@
 F 0 "C10" H 3500 4400 50  0000 L CNN
 F 1 "0.1µF" H 3500 4300 50  0000 L CNN
-F 2 "Capacitor_SMD:C_0201_0603Metric" H 3888 4250 50  0001 C CNN
+F 2 "Capacitor_SMD:C_0402_1005Metric" H 3888 4250 50  0001 C CNN
 F 3 "~" H 3850 4400 50  0001 C CNN
 	1    3850 4400
@@
 F 0 "C7" H 3000 4400 50  0000 L CNN
 F 1 "4.7µF" H 3000 4300 50  0000 L CNN
-F 2 "Capacitor_SMD:C_0201_0603Metric" H 3388 4250 50  0001 C CNN
+F 2 "Capacitor_SMD:C_0402_1005Metric" H 3388 4250 50  0001 C CNN
 F 3 "~" H 3350 4400 50  0001 C CNN
 	1    3350 4400
@@
 F 0 "C17" V 8050 1000 50  0000 L CNN
 F 1 "100nF" V 7950 900 50  0000 L CNN
-F 2 "Capacitor_SMD:C_0201_0603Metric" H 7888 700 50  0001 C CNN
+F 2 "Capacitor_SMD:C_0402_1005Metric" H 7888 700 50  0001 C CNN
 F 3 "~" H 7850 850 50  0001 C CNN
 	1    7850 850
@@
 F 0 "C9" H 3350 650 50  0000 L CNN
 F 1 "0.1µF" H 3350 550 50  0000 L CNN
-F 2 "Capacitor_SMD:C_0201_0603Metric" H 3738 500 50  0001 C CNN
+F 2 "Capacitor_SMD:C_0402_1005Metric" H 3738 500 50  0001 C CNN
 F 3 "~" H 3700 650 50  0001 C CNN
 	1    3700 650
@@
 F 0 "C2" V 800 2450 50  0000 L CNN
 F 1 "1µF" V 800 2200 50  0000 L CNN
-F 2 "Capacitor_SMD:C_0201_0603Metric" H 988 2250 50  0001 C CNN
+F 2 "Capacitor_SMD:C_0402_1005Metric" H 988 2250 50  0001 C CNN
 F 3 "~" H 950 2400 50  0001 C CNN
 	1    950  2400
@@
 F 0 "R7" H 1300 6600 50  0000 L CNN
 F 1 "10K" H 1300 6500 50  0000 L CNN
-F 2 "Resistor_SMD:R_0201_0603Metric" V 1180 6550 50  0001 C CNN
+F 2 "Resistor_SMD:R_0402_1005Metric" V 1180 6550 50  0001 C CNN
 F 3 "~" H 1250 6550 50  0001 C CNN
 	1    1250 6550
@@
 F 0 "C22" V 8050 2200 50  0000 L CNN
 F 1 "100nF" V 7950 2100 50  0000 L CNN
-F 2 "Capacitor_SMD:C_0201_0603Metric" H 7888 1900 50  0001 C CNN
+F 2 "Capacitor_SMD:C_0402_1005Metric" H 7888 1900 50  0001 C CNN
 F 3 "~" H 7850 2050 50  0001 C CNN
 	1    7850 2050

Commit message: Board: Adjustments
Parts:
- removed C1, C12: 10µF, Capacitor_SMD:C_0805_2012Metric, symbol Device:C
- removed C10, C5: 0.1µF, Capacitor_SMD:C_0402_1005Metric, symbol Device:C
- removed C11, C13, C8: 22µF, Capacitor_SMD:C_0805_2012Metric, symbol Device:C
- removed C3: 220nF, Capacitor_SMD:C_0805_2012Metric, symbol Device:C
- removed C4: 1µF, Capacitor_SMD:C_0402_1005Metric, symbol Device:C
- removed C7: 4.7µF, Capacitor_SMD:C_0402_1005Metric, symbol Device:C
- removed D4, D5: D_Schottky, Diode_SMD:D_SMA, symbol Device:D_Schottky
- removed D6: SP0503BAHT, Package_TO_SOT_SMD:SOT-143, symbol Power_Protection:SP0503BAHT
- removed J2: USB_C_Receptacle_USB2.0, USB_C_Receptacle_JAE_DX07S016JA1:USB_C_Receptacle_JAE_DX07S016JA1, symbol Connector:USB_C_Receptacle_USB2.0
- removed JP1: SolderJumper_2_Bridged, Jumper:SolderJumper-2_P1.3mm_Bridged_RoundedPad1.0x1.5mm, symbol Jumper:SolderJumper_2_Bridged
- removed JP4: Jumper_NO_Small, Connector_PinHeader_2.54mm:PinHeader_1x02_P2.54mm_Vertical, symbol Device:Jumper_NO_Small
- removed L1: 2.2µH, TDK_SPM5030:TDK_SPM5030, symbol Device:L
- removed R12, R9: 100K, Resistor_SMD:R_0402_1005Metric, symbol Device:R
- removed R13: 24.9K, Resistor_SMD:R_0402_1005Metric, symbol Device:R
- removed R14: 1K, Resistor_SMD:R_0402_1005Metric, symbol Device:R
- removed R15, R16: 5.1K, Resistor_SMD:R_0402_1005Metric, symbol Device:R
- removed R7: 10K, Resistor_SMD:R_0402_1005Metric, symbol Device:R
- removed R8: 866K, Resistor_SMD:R_0402_1005Metric, symbol Device:R
- removed U1: LMR33630BDDA, Package_SO:Texas_HSOP-8-1EP_3.9x4.9mm_P1.27mm_ThermalVias, symbol Regulator_Switching:LMR33630BDDA
- removed U3: AZ1117C-3.3, Package_TO_SOT_SMD:SOT-89-3, symbol Regulator_Linear:AZ1117-3.3
- removed U4: CP2102N-A01-GQFN24, Package_DFN_QFN:QFN-24-1EP_4x4mm_P0.5mm_EP2.6x2.6mm, symbol Interface_USB:CP2102N-A01-GQFN24
- added J8, J9: Conn_01x04_Male, Connector_PinHeader_2.54mm:PinHeader_1x04_P2.54mm_Vertical, symbol Connector:Conn_01x04_Male
- added Q1, Q2: BC817, Package_TO_SOT_SMD:SOT-23, symbol Transistor_BJT:BC817
- added R23, R24: 10K, Resistor_SMD:R_0402_1005Metric, symbol Device:R
- C15: value 0.47µF -> 0.47uF
- C16, C18, C19, C20, C21, C9: value 0.1µF -> 0.1uF
- C2: value 1µF -> 1uF
- C6: value 10µF -> 10uF
- R1, R2: footprint Resistor_SMD:R_0402_1005Metric -> Resistor_SMD:R_0603_1608Metric
- R4, R5: value 65R -> 64.9R
- R6: value 5R -> 4.99R
- U7: value MCP2562-E-MF -> MCP2562FD-E-MF
Connections:
- net labels removed: +5VA, USB_D+, USB_D-
- wire segments 105 -> 57
Other:
- moved on the sheet: C14, C15, C16, C17, C18, C19, C20, C21, C22, C6, C9, J4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
